File: Tim/tic_tac_toe_wire.brd (EAGLE design)
At the start: 53.3 x 52.7 mm, 18 parts, among them IC1 PCF8574P, U1 ATMEGA328P_PDIP

Commit message: 3 try
Parts:
- moved U1 3.18 mm to (15.2, 19.7)
- moved JP2 2.62 mm to (22.2, 3.81)
- moved IC2 1.91 mm to (9.53, 43.2)
Connections:
- removed net N$15: IC1.12, LD9.AX
- removed net N$16: IC1.11, LD9.AR
- removed net N$17: IC1.10, LD6.AR
- removed net N$18: IC1.9, LD6.AX
- removed net N$19: IC1.7, LD3.AR
- removed net N$20: IC1.6, LD3.AX
- removed net N$21: IC1.5, LD8.AX
- removed net N$22: IC1.4, LD8.AR
- removed net N$23: LD7.AX, U1.18
- removed net N$24: LD7.AR, U1.17
- removed net N$25: LD4.AR, U1.16
- removed net N$26: LD4.AX, U1.13
- removed net N$27: LD1.AR, U1.12
- removed net N$28: LD1.AX, U1.11
- removed net N$29: LD5.AR, U1.6
- removed net N$30: LD5.AX, U1.5
- removed net N$31: LD2.AX, U1.23
- removed net N$32: LD2.AR, U1.24
- net N$2: now also U1.5; no longer U1.14
- net N$3: now also U1.6; no longer U1.15
Routing:
- net N$22: track 67.3 -> 0.00 mm
- net N$32: track 66.5 -> 0.00 mm
- net N$18: track 63.8 -> 0.00 mm
- net N$25: track 62.2 -> 0.00 mm
- net N$29: track 60.2 -> 0.00 mm
- net N$3: track 86.4 -> 37.5 mm
- net GND: track 219.0 -> 171.0 mm
- net N$31: track 45.3 -> 0.00 mm
- net N$16: track 44.1 -> 0.00 mm
- net N$15: track 41.6 -> 0.00 mm
- net N$24: track 32.3 -> 0.00 mm
- net N$30: track 32.1 -> 0.00 mm
- net N$17: track 27.1 -> 0.00 mm
- net N$21: track 26.8 -> 0.00 mm
- net N$23: track 26.0 -> 0.00 mm
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Other:
- board size 53.3 x 52.7 mm -> 52.7 x 51.4 mm
