File: Tim/tic_tac_toe_wire.sch (EAGLE design)
At the start: 18 parts, among them IC1 PCF8574P, U1 ATMEGA328P_PDIP

Commit message: 3 try
Connections:
- removed net N$15: IC1.P7, LD9.AG
- removed net N$16: IC1.P6, LD9.AR
- removed net N$17: IC1.P5, LD6.AR
- removed net N$18: IC1.P4, LD6.AG
- removed net N$19: IC1.P3, LD3.AR
- removed net N$20: IC1.P2, LD3.AG
- removed net N$21: IC1.P1, LD8.AG
- removed net N$22: IC1.P0, LD8.AR
- removed net N$23: LD7.AG, U1.PB4(MISO)
- removed net N$24: LD7.AR, U1.PB3(MOSI/OC2)
- removed net N$25: LD4.AR, U1.PB2(SS/OC1B)
- removed net N$26: LD4.AG, U1.PD7(AIN1)
- removed net N$27: LD1.AR, U1.PD6(AIN0)
- removed net N$28: LD1.AG, U1.PD5(T1)
- removed net N$29: LD5.AR, U1.PD4(XCK/T0)
- removed net N$30: LD5.AG, U1.PD3(INT1)
- removed net N$31: LD2.AG, U1.PC0(ADC0)
- removed net N$32: LD2.AR, U1.PC1(ADC1)
- net N$2: now also U1.PD3(INT1); no longer U1.PB0(ICP)
- net N$3: now also U1.PD4(XCK/T0); no longer U1.PB1(OC1A)
Other:
- moved on the sheet: IC1
