File: Cyrill/tictactoe19_11.sch (EAGLE design)
At the start: 18 parts, among them IC1 PCF8574P, U1 ATMEGA328P_PDIP

Commit message: next try :P
Connections:
- removed net GND2: IC2.3, IC2.5, S2.3, S2.4, S3.3, S3.4, U1.GND@1
- removed net N$30: LD5.AG
- removed net N$7: IC1.A0, IC1.A1, IC1.A2, IC1.VSS
- new net N$29: LD5.AG, U1.PC3(ADC3)
- net GND: now also IC1.A0, IC1.A1, IC1.A2, IC1.VSS, IC2.3, IC2.5, S2.3, S2.4, S3.3, S3.4, U1.GND@1
- net N$11: now also U1.PD4(XCK/T0); no longer U1.PD2(INT0)
- net VCC: now also IC1.VDD, U1.AVCC
