File: Cyrill/tictactoe19_11.brd (EAGLE design)
At the start: 69.5 x 67.3 mm, 18 parts, among them IC1 PCF8574P, U1 ATMEGA328P_PDIP

Commit message: X
Connections:
- net N$30: no longer U1.26
Routing:
- net N$30: track 69.8 -> 50.8 mm
Changed lines of the file:
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@@
 <signal name="N$30">
 <contactref element="LD5" pad="AX"/>
-<contactref element="U1" pad="26"/>
-<wire x1="11.43" y1="16.51" x2="11.43" y2="35.56" width="0.4064" layer="16"/>
 <wire x1="11.43" y1="35.56" x2="20.32" y2="35.56" width="0.4064" layer="16"/>
 <wire x1="20.32" y1="35.56" x2="20.32" y2="40.64" width="0.4064" layer="16"/>

Commit message: next try :P
Parts:
- moved S2 4.02 mm to (54.6, 21.6)
- moved S3 3.81 mm to (66.0, 21.6)
- moved IC2 2.84 mm to (57.1, 6.35)
- moved JP3 2.84 mm to (21.6, 1.27)
- moved LD2 1.27 mm to (64.8, 45.7)
- moved LD5 1.27 mm to (55.9, 45.7)
- moved LD8 1.27 mm to (45.7, 45.7)
Connections:
- removed net GND2: IC2.3, IC2.5, S2.3, S2.4, S3.3, S3.4, U1.8
- removed net N$30: LD5.AX
- removed net N$7: IC1.1, IC1.2, IC1.3, IC1.8
- removed net VDD: IC1.16
- new net N$29: LD5.AX, U1.26
- net GND: now also IC1.1, IC1.2, IC1.3, IC1.8, IC2.3, IC2.5, S2.3, S2.4, S3.3, S3.4, U1.8
- net N$11: now also U1.6; no longer U1.4
- net VCC: now also IC1.16, U1.20
Routing:
- net GND: track 48.7 -> 290.1 mm
- net GND2: track 101.2 -> 0.00 mm
- net N$29: track 0.00 -> 71.1 mm
- net VCC: track 229.9 -> 281.9 mm
- net N$30: track 50.8 -> 0.00 mm
- net N$7: track 25.4 -> 0.00 mm
- net N$11: track 6.35 -> 12.7 mm
- net N$13: track 57.6 -> 63.2 mm
- net N$14: track 49.3 -> 54.3 mm
- net N$12: track 47.0 -> 50.8 mm
- net N$1: track 44.5 -> 48.3 mm
- net N$19: track 86.4 -> 89.4 mm
- net N$8: track 25.4 -> 27.9 mm
- net N$6: track 59.7 -> 62.2 mm
- net N$20: track 83.8 -> 85.1 mm
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
Commit message: ...
Other:
- board size 69.5 x 67.3 mm -> 69.5 x 68.6 mm
Changed lines of the file:
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@@
 <board>
 <plain>
-<wire x1="3.81" y1="-2.54" x2="73.33" y2="-2.54" width="0" layer="20"/>
-<wire x1="73.33" y1="-2.54" x2="73.33" y2="64.76" width="0" layer="20"/>
+<wire x1="3.81" y1="-3.81" x2="73.33" y2="-3.81" width="0" layer="20"/>
+<wire x1="73.33" y1="-3.81" x2="73.33" y2="64.76" width="0" layer="20"/>
 <wire x1="73.33" y1="64.76" x2="3.81" y2="64.76" width="0" layer="20"/>
-<wire x1="3.81" y1="64.76" x2="3.81" y2="-2.54" width="0" layer="20"/>
+<wire x1="3.81" y1="64.76" x2="3.81" y2="-3.81" width="0" layer="20"/>
 </plain>
 <attributes>

Commit message: bla
Parts:
- moved JP2 1.27 mm to (6.35, 5.08)
- moved JP3 1.27 mm to (21.6, 0.00)
Routing:
- net VCC: track 281.9 -> 271.8 mm
- net N$10: track 20.8 -> 27.4 mm
- net GND: track 290.1 -> 296.5 mm
- net N$21: track 87.6 -> 82.6 mm
- net N$22: track 55.9 -> 53.3 mm
- net N$24: track 64.8 -> 62.2 mm
- net N$23: track 61.0 -> 58.4 mm
- net N$5: track 5.08 -> 3.81 mm
- net N$4: track 5.08 -> 3.81 mm
- net N$2: track 5.08 -> 3.81 mm
- net N$11: track 12.7 -> 14.0 mm
- net N$19: track 89.4 -> 90.2 mm
- added copper zone on layer 16, net N$7
Other:
- board size 69.5 x 68.6 mm -> 70.8 x 66 mm

Commit message: frei_final
Parts:
- moved LD9 2.84 mm to (47.0, 55.9)
- moved LD3 2.54 mm to (64.8, 55.9)
- moved LD6 2.54 mm to (55.9, 55.9)
- moved LD7 1.27 mm to (47.0, 35.6)
- moved LD8 1.27 mm to (47.0, 45.7)
Routing:
- net N$10: track 27.4 -> 20.8 mm
- net VCC: track 271.8 -> 276.2 mm
- net N$25: track 35.6 -> 39.4 mm
- net N$26: track 27.9 -> 31.8 mm
- net N$21: track 82.6 -> 85.1 mm
- net N$24: track 62.2 -> 64.8 mm
- net N$23: track 58.4 -> 61.0 mm
- net N$22: track 53.3 -> 55.9 mm
- net N$27: track 25.4 -> 26.7 mm
- net N$18: track 45.7 -> 47.0 mm
Other:
- board size 70.8 x 66 mm -> 70.8 x 69.8 mm

Commit message: final2
Parts:
- moved LD7 2.54 mm to (44.5, 35.6)
- moved LD8 2.54 mm to (44.5, 45.7)
- moved LD9 2.54 mm to (44.5, 55.9)
- moved LD4 1.27 mm to (54.6, 35.6)
- moved LD5 1.27 mm to (54.6, 45.7)
- moved LD6 1.27 mm to (54.6, 55.9)
Routing:
- net N$27: track 26.7 -> 24.1 mm
- net N$26: track 31.8 -> 29.2 mm
- net N$25: track 39.4 -> 36.8 mm
- net N$18: track 47.0 -> 44.4 mm
- net N$15: track 48.6 -> 46.0 mm
- net VCC: track 276.2 -> 278.1 mm
- net N$28: track 33.3 -> 31.8 mm
- net N$29: track 71.1 -> 69.8 mm
- net N$16: track 43.2 -> 41.9 mm
- net N$22: track 55.9 -> 54.6 mm
- net N$31: track 73.7 -> 72.4 mm
- net N$23: track 61.0 -> 59.7 mm
- net N$17: track 40.6 -> 39.4 mm
Other:
- board size 70.8 x 69.8 mm -> 69.5 x 68.6 mm
- board text added: "DonFrei"

Commit message: final3
Routing:
- net N$15: track 46.0 -> 47.0 mm
Changed lines of the file:
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@@
 <contactref element="LD7" pad="AR"/>
 <contactref element="U1" pad="23"/>
-<wire x1="46.99" y1="35.56" x2="45.72" y2="33.02" width="0.4064" layer="16"/>
-<wire x1="45.72" y1="33.02" x2="26.67" y2="33.02" width="0.4064" layer="16"/>
+<wire x1="46.99" y1="35.56" x2="46.99" y2="33.02" width="0.4064" layer="16"/>
+<wire x1="46.99" y1="33.02" x2="26.67" y2="33.02" width="0.4064" layer="16"/>
 <wire x1="26.67" y1="33.02" x2="26.67" y2="25.4" width="0.4064" layer="16"/>
 <wire x1="26.67" y1="25.4" x2="19.05" y2="25.4" width="0.4064" layer="16"/>
@@
 <vertex x="2.54" y="64.77"/>
 <vertex x="72.39" y="64.77"/>
-<vertex x="73.66" y="-3.81"/>
+<vertex x="72.39" y="-3.81"/>
 <vertex x="2.54" y="-3.81"/>
 </polygon>
