File: Andreas/tic_tac_toe_board/version2/my_tic_tac_toe_board2.brd (EAGLE design)
At the start: 54.3 x 80 mm, 18 parts, among them IC1 PCF8574P, U1 ATMEGA328P_PDIP

Commit message: andu final solution
Connections:
- net S$19 renamed S$2
Routing:
- net N$9: track 137.2 -> 141.0 mm
- net N$2: track 253.0 -> 253.8 mm
- net S$5: track 34.8 -> 35.6 mm
- net S$2: track 54.9 -> 55.7 mm
- added copper zone on layer 16, net S$19
- added copper zone on layer 1, net S$21
