File: Rico/tic-tac-toe.brd (EAGLE design)
At the start: 56.8 x 66 mm, 18 parts, among them IC1 PCF8574P, U1 ATMEGA328P_PDIP

Commit message: ricoh: final version -> bestellen
Parts:
- moved JP3 3.81 mm to (52.1, 36.8)
Connections:
- removed net S$1: IC1.13
Routing:
- net S$10: track 94.3 -> 90.5 mm
- net S$1: track 3.81 -> 0.00 mm
- net GND: track 175.7 -> 171.8 mm
- net S$21: track 40.9 -> 39.9 mm
- net S$18: track 55.4 -> 54.4 mm
- added copper zone on layer 16, net S$1
Other:
- board size 56.8 x 66 mm -> 56.8 x 64.8 mm
Changed lines of the file:
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@@
 <plain>
 <wire x1="44.45" y1="12.7" x2="101.27" y2="12.7" width="0" layer="20"/>
-<wire x1="101.27" y1="12.7" x2="101.27" y2="78.73" width="0" layer="20"/>
-<wire x1="101.27" y1="78.73" x2="44.45" y2="78.73" width="0" layer="20"/>
-<wire x1="44.45" y1="78.73" x2="44.45" y2="12.7" width="0" layer="20"/>
+<wire x1="101.27" y1="12.7" x2="101.27" y2="77.46" width="0" layer="20"/>
+<wire x1="101.27" y1="77.46" x2="44.45" y2="77.46" width="0" layer="20"/>
+<wire x1="44.45" y1="77.46" x2="44.45" y2="12.7" width="0" layer="20"/>
 </plain>
 <attributes>
@@
 </class>
 </classes>
-<designrules name="default">
+<designrules name="bastli">
 <description language="de">&lt;b&gt;EAGLE Design Rules&lt;/b&gt;
 &lt;p&gt;
@@
 <param name="mtCopper" value="0.035mm 0.035mm 0.035mm 0.035mm 0.035mm 0.035mm 0.035mm 0.035mm 0.035mm 0.035mm 0.035mm 0.035mm 0.035mm 0.035mm 0.035mm 0.035mm"/>
 <param name="mtIsolate" value="1.5mm 0.15mm 0.2mm 0.15mm 0.2mm 0.15mm 0.2mm 0.15mm 0.2mm 0.15mm 0.2mm 0.15mm 0.2mm 0.15mm 0.2mm"/>
-<param name="mdWireWire" value="8mil"/>
-<param name="mdWirePad" value="8mil"/>
-<param name="mdWireVia" value="8mil"/>
-<param name="mdPadPad" value="8mil"/>
-<param name="mdPadVia" value="8mil"/>
-<param name="mdViaVia" value="8mil"/>
-<param name="mdSmdPad" value="8mil"/>
-<param name="mdSmdVia" value="8mil"/>
-<param name="mdSmdSmd" value="8mil"/>
+<param name="mdWireWire" value="0.4mm"/>
+<param name="mdWirePad" value="0.4mm"/>
+<param name="mdWireVia" value="0.4mm"/>
+<param name="mdPadPad" value="0.4mm"/>
+<param name="mdPadVia" value="0.4mm"/>
+<param name="mdViaVia" value="0.4mm"/>
+<param name="mdSmdPad" value="0.4mm"/>
+<param name="mdSmdVia" value="0.4mm"/>
+<param name="mdSmdSmd" value="0.4mm"/>
 <param name="mdViaViaSameLayer" value="8mil"/>
 <param name="mnLayersViaInSmd" value="2"/>
-<param name="mdCopperDimension" value="40mil"/>
-<param name="mdDrill" value="8mil"/>
+<param name="mdCopperDimension" value="0.4mm"/>
+<param name="mdDrill" value="0.4mm"/>
 <param name="mdSmdStop" value="0mil"/>
-<param name="msWidth" value="10mil"/>
-<param name="msDrill" value="24mil"/>
+<param name="msWidth" value="0.4mm"/>
+<param name="msDrill" value="0.1mm"/>
 <param name="msMicroVia" value="9.99mm"/>
 <param name="msBlindViaRatio" value="0.5"/>
@@
 <pass name="Default">
 <param name="RoutingGrid" value="50mil"/>
-<param name="tpViaShape" value="round"/>
+<param name="tpViaShape" value="octagon"/>
 <param name="PrefDir.1" value="|"/>
 <param name="PrefDir.2" value="0"/>
@@
 <pass name="Route" refer="Default" active="yes">
 </pass>
-<pass name="Optimize1" refer="Default" active="yes">
+<pass name="Optimize1" refer="Default" active="no">
 <param name="cfVia" value="99"/>
 <param name="cfExtdStep" value="10"/>
@@
 <param name="mnRipupLevel" value="0"/>
 </pass>
-<pass name="Optimize2" refer="Optimize1" active="yes">
+<pass name="Optimize2" refer="Optimize1" active="no">
 <param name="cfNonPref" value="0"/>
 <param name="cfChangeDir" value="6"/>
@@
 <param name="cfHugging" value="0"/>
 </pass>
-<pass name="Optimize3" refer="Optimize2" active="yes">
+<pass name="Optimize3" refer="Optimize2" active="no">
 <param name="cfChangeDir" value="8"/>
 <param name="cfPadImpact" value="0"/>
 <param name="cfSmdImpact" value="0"/>
 </pass>
-<pass name="Optimize4" refer="Optimize3" active="yes">
+<pass name="Optimize4" refer="Optimize3" active="no">
 <param name="cfChangeDir" value="25"/>
 </pass>
@@
 <element name="JP1" library="SparkFun-Connectors" package="1X02" value="M02PTH" x="78.74" y="27.94"/>
 <element name="JP2" library="SparkFun-Connectors" package="1X03" value="" x="63.5" y="27.94"/>
-<element name="JP3" library="SparkFun-Connectors" package="1X04" value="" x="48.26" y="36.83" rot="R270"/>
+<element name="JP3" library="SparkFun-Connectors" package="1X04" value="" x="52.07" y="36.83" rot="R270"/>
 <element name="IC2" library="ic-package" package="SOCKET-08" value="" x="92.71" y="21.59" rot="R180"/>
 </elements>
@@
 <wire x1="78.74" y1="38.1" x2="77.47" y2="36.83" width="0.4064" layer="16"/>
 <wire x1="77.47" y1="36.83" x2="68.58" y2="36.83" width="0.4064" layer="16"/>
-<wire x1="48.26" y1="36.83" x2="60.96" y2="36.83" width="0.4064" layer="16"/>
+<wire x1="52.07" y1="36.83" x2="60.96" y2="36.83" width="0.4064" layer="16"/>
 <wire x1="60.96" y1="36.83" x2="66.04" y2="36.83" width="0.4064" layer="16"/>
 <wire x1="66.04" y1="36.83" x2="67.31" y2="38.1" width="0.4064" layer="16"/>
@@
 <wire x1="76.4794" y1="22.5806" x2="76.2" y2="22.86" width="0.4064" layer="16"/>
 <contactref element="S2" pad="1"/>
-<wire x1="76.4794" y1="22.5806" x2="76.7588" y2="22.5806" width="0" layer="19" extent="16-16"/>
 <wire x1="76.7588" y1="22.5806" x2="76.7588" y2="22.3012" width="0.4064" layer="16"/>
 <wire x1="76.7588" y1="22.3012" x2="76.4794" y2="22.5806" width="0.4064" layer="16"/>
@@
 <contactref element="JP2" pad="2"/>
 <wire x1="66.04" y1="27.94" x2="66.04" y2="31.75" width="0.4064" layer="16"/>
-</signal>
-<signal name="S$1">
-<contactref element="IC1" pad="13"/>
-<wire x1="49.53" y1="53.34" x2="45.72" y2="53.34" width="0.4064" layer="1"/>
 </signal>
 <signal name="S$3">
@@
 <contactref element="IC1" pad="10"/>
 <wire x1="68.58" y1="72.39" x2="68.58" y2="74.93" width="0.4064" layer="16"/>
-<wire x1="68.58" y1="74.93" x2="67.31" y2="76.2" width="0.4064" layer="16"/>
-<wire x1="67.31" y1="76.2" x2="48.26" y2="76.2" width="0.4064" layer="16"/>
-<wire x1="48.26" y1="76.2" x2="46.99" y2="74.93" width="0.4064" layer="16"/>
+<wire x1="68.58" y1="74.93" x2="46.99" y2="74.93" width="0.4064" layer="16"/>
 <wire x1="46.99" y1="74.93" x2="46.99" y2="62.23" width="0.4064" layer="16"/>
 <wire x1="46.99" y1="62.23" x2="48.26" y2="60.96" width="0.4064" layer="16"/>
@@
 <wire x1="48.26" y1="58.42" x2="45.72" y2="60.96" width="0.4064" layer="16"/>
 <wire x1="45.72" y1="60.96" x2="45.72" y2="76.2" width="0.4064" layer="16"/>
-<wire x1="45.72" y1="76.2" x2="46.99" y2="77.47" width="0.4064" layer="16"/>
-<wire x1="46.99" y1="77.47" x2="74.93" y2="77.47" width="0.4064" layer="16"/>
-<wire x1="74.93" y1="77.47" x2="76.2" y2="76.2" width="0.4064" layer="16"/>
+<wire x1="45.72" y1="76.2" x2="76.2" y2="76.2" width="0.4064" layer="16"/>
 <wire x1="76.2" y1="76.2" x2="76.2" y2="72.39" width="0.4064" layer="16"/>
 </signal>
@@
 <contactref element="JP3" pad="4"/>
 <contactref element="U1" pad="11"/>
-<wire x1="48.26" y1="29.21" x2="48.26" y2="17.78" width="0.4064" layer="16"/>
-<wire x1="48.26" y1="17.78" x2="52.07" y2="13.97" width="0.4064" layer="16"/>
-<wire x1="52.07" y1="13.97" x2="100.33" y2="13.97" width="0.4064" layer="16"/>
+<wire x1="52.07" y1="29.21" x2="52.07" y2="17.78" width="0.4064" layer="16"/>
+<wire x1="52.07" y1="17.78" x2="55.88" y2="13.97" width="0.4064" layer="16"/>
+<wire x1="55.88" y1="13.97" x2="100.33" y2="13.97" width="0.4064" layer="16"/>
 <wire x1="100.33" y1="13.97" x2="100.33" y2="29.21" width="0.4064" layer="16"/>
 <wire x1="100.33" y1="29.21" x2="88.9" y2="29.21" width="0.4064" layer="16"/>
 <wire x1="88.9" y1="29.21" x2="88.9" y2="31.75" width="0.4064" layer="16"/>
 </signal>
+<signal name="S$1">
+<polygon width="0.4064" layer="16">
+<vertex x="44.45" y="77.47"/>
+<vertex x="101.6" y="77.47"/>
+<vertex x="101.6" y="12.7"/>
+<vertex x="44.45" y="12.7"/>
+</polygon>
+</signal>
 </signals>
