File: Donjan/tictactoe2.brd (EAGLE design)
At the start: 53 x 63.5 mm, 18 parts, among them IC1 PCF8574P, U1 ATMEGA328P_PDIP

Commit message: version 2 (fixes)  and a more compact one
Parts:
- moved JP3 39.0 mm to (35.6, 49.5), turned to 90 degrees
Connections:
- net N$9 renamed S$19
Routing:
- net GND: track 138.6 -> 170.9 mm
- net S$19: track 23.0 -> 29.2 mm
- net S$11: track 46.4 -> 45.1 mm
- net S$10: track 69.2 -> 67.9 mm
- net S$14: track 43.8 -> 42.7 mm
Other:
- board size 53 x 63.5 mm -> 50.5 x 63.5 mm
Changed lines of the file:
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@@
 <board>
 <plain>
-<wire x1="0.635" y1="1.905" x2="53.645" y2="1.905" width="0" layer="20"/>
-<wire x1="53.645" y1="1.905" x2="53.645" y2="65.395" width="0" layer="20"/>
-<wire x1="53.645" y1="65.395" x2="0.635" y2="65.395" width="0" layer="20"/>
+<wire x1="0.635" y1="1.905" x2="51.105" y2="1.905" width="0" layer="20"/>
+<wire x1="51.105" y1="1.905" x2="51.105" y2="65.395" width="0" layer="20"/>
+<wire x1="51.105" y1="65.395" x2="0.635" y2="65.395" width="0" layer="20"/>
 <wire x1="0.635" y1="65.395" x2="0.635" y2="1.905" width="0" layer="20"/>
-<dimension x1="5.715" y1="61.595" x2="25.4" y2="61.595" x3="15.5575" y3="71.755" textsize="1.778" layer="1" dtype="horizontal"/>
-<dimension x1="25.4" y1="61.595" x2="45.085" y2="61.595" x3="35.2425" y3="71.755" textsize="1.778" layer="1" dtype="horizontal"/>
-<dimension x1="45.085" y1="61.595" x2="45.085" y2="46.355" x3="62.23" y3="53.975" textsize="1.778" layer="1" dtype="horizontal"/>
-<dimension x1="45.085" y1="46.355" x2="45.085" y2="31.115" x3="62.23" y3="38.735" textsize="1.778" layer="1" dtype="horizontal"/>
-<circle x="10.16" y="48.26" radius="1.79605" width="0.4064" layer="1"/>
-<circle x="10.16" y="31.115" radius="2.00804375" width="0.4064" layer="1"/>
-<circle x="36.83" y="1.905" radius="1.419903125" width="0.4064" layer="1"/>
-<circle x="0.635" y="3.81" radius="1.419903125" width="0.4064" layer="1"/>
-<circle x="6.985" y="1.905" radius="1.419903125" width="0.4064" layer="1"/>
 </plain>
 <attributes>
@@
 <element name="JP2" library="SparkFun-Connectors" package="1X03" value="" x="6.35" y="14.605"/>
 <element name="IC2" library="ic-package" package="SOCKET-08" value="" x="37.465" y="7.62" rot="R270"/>
-<element name="JP3" library="SparkFun-Connectors" package="1X04" value="" x="48.26" y="12.7" rot="R270"/>
+<element name="JP3" library="SparkFun-Connectors" package="1X04" value="" x="35.56" y="49.53" rot="R90"/>
 </elements>
 <signals>
@@
 <wire x1="19.685" y1="34.29" x2="17.145" y2="34.29" width="0.4064" layer="16"/>
 <wire x1="19.685" y1="31.75" x2="17.145" y2="31.75" width="0.4064" layer="16"/>
-<wire x1="41.275" y1="3.81" x2="48.26" y2="3.81" width="0.4064" layer="16"/>
-<wire x1="48.26" y1="3.81" x2="48.26" y2="5.08" width="0.4064" layer="16"/>
 <wire x1="17.145" y1="31.75" x2="17.145" y2="29.845" width="0.4064" layer="16"/>
 <wire x1="17.145" y1="29.845" x2="19.05" y2="29.845" width="0.4064" layer="16"/>
@@
 <wire x1="28.2956" y1="10.2362" x2="27.94" y2="9.525" width="0.4064" layer="16"/>
 <wire x1="27.94" y1="9.525" x2="27.94" y2="8.255" width="0.4064" layer="16"/>
+<wire x1="35.56" y1="57.15" x2="33.02" y2="57.15" width="0.4064" layer="16"/>
+<wire x1="33.02" y1="57.15" x2="33.02" y2="24.13" width="0.4064" layer="16"/>
+<wire x1="33.02" y1="24.13" x2="27.94" y2="24.13" width="0.4064" layer="16"/>
 </signal>
 <signal name="VCC">
@@
 <wire x1="29.845" y1="11.43" x2="31.75" y2="11.43" width="0.4064" layer="16"/>
 </signal>
-<signal name="N$9">
-<contactref element="U1" pad="11"/>
-<contactref element="JP3" pad="1"/>
-<wire x1="33.02" y1="13.97" x2="48.895" y2="13.97" width="0.4064" layer="16"/>
-<wire x1="48.895" y1="13.97" x2="48.26" y2="12.7" width="0.4064" layer="16"/>
-<wire x1="31.75" y1="18.415" x2="31.75" y2="16.51" width="0.4064" layer="16"/>
-<wire x1="31.75" y1="16.51" x2="33.02" y2="16.51" width="0.4064" layer="16"/>
-<wire x1="33.02" y1="16.51" x2="33.02" y2="13.97" width="0.4064" layer="16"/>
-</signal>
 <signal name="N$10">
 <contactref element="U1" pad="27"/>
@@
 <contactref element="LD3" pad="AR"/>
 <wire x1="34.29" y1="18.415" x2="34.29" y2="15.24" width="0.4064" layer="16"/>
-<wire x1="34.29" y1="15.24" x2="50.8" y2="15.24" width="0.4064" layer="16"/>
-<wire x1="50.8" y1="15.24" x2="50.8" y2="61.595" width="0.4064" layer="16"/>
-<wire x1="50.8" y1="61.595" x2="47.625" y2="61.595" width="0.4064" layer="16"/>
+<wire x1="34.29" y1="15.24" x2="50.165" y2="15.24" width="0.4064" layer="16"/>
+<wire x1="50.165" y1="15.24" x2="50.165" y2="61.595" width="0.4064" layer="16"/>
+<wire x1="50.165" y1="61.595" x2="47.625" y2="61.595" width="0.4064" layer="16"/>
 </signal>
 <signal name="S$11">
@@
 <contactref element="LD8" pad="AR"/>
 <wire x1="36.83" y1="18.415" x2="36.83" y2="16.51" width="0.4064" layer="16"/>
-<wire x1="36.83" y1="16.51" x2="49.53" y2="16.51" width="0.4064" layer="16"/>
-<wire x1="49.53" y1="16.51" x2="49.53" y2="46.355" width="0.4064" layer="16"/>
-<wire x1="49.53" y1="46.355" x2="47.625" y2="46.355" width="0.4064" layer="16"/>
+<wire x1="36.83" y1="16.51" x2="48.895" y2="16.51" width="0.4064" layer="16"/>
+<wire x1="48.895" y1="16.51" x2="48.895" y2="46.355" width="0.4064" layer="16"/>
+<wire x1="48.895" y1="46.355" x2="47.625" y2="46.355" width="0.4064" layer="16"/>
 </signal>
 <signal name="S$12">
@@
 <contactref element="LD2" pad="AR"/>
 <contactref element="U1" pad="18"/>
-<wire x1="31.75" y1="26.035" x2="31.75" y2="61.595" width="0.4064" layer="16"/>
-<wire x1="31.75" y1="61.595" x2="27.94" y2="61.595" width="0.4064" layer="16"/>
+<wire x1="31.75" y1="26.035" x2="31.75" y2="50.165" width="0.4064" layer="16"/>
+<wire x1="31.75" y1="50.165" x2="27.94" y2="50.165" width="0.4064" layer="16"/>
+<wire x1="27.94" y1="50.165" x2="27.94" y2="61.595" width="0.4064" layer="16"/>
 </signal>
 <signal name="S$14">
 <contactref element="LD3" pad="AX"/>
 <contactref element="U1" pad="17"/>
-<wire x1="34.29" y1="26.035" x2="34.29" y2="61.595" width="0.4064" layer="16"/>
-<wire x1="34.29" y1="61.595" x2="42.545" y2="61.595" width="0.4064" layer="16"/>
+<wire x1="34.29" y1="26.035" x2="34.29" y2="39.37" width="0.4064" layer="16"/>
+<wire x1="34.29" y1="39.37" x2="40.64" y2="39.37" width="0.4064" layer="16"/>
+<wire x1="40.64" y1="39.37" x2="40.64" y2="48.895" width="0.4064" layer="16"/>
+<wire x1="40.64" y1="48.895" x2="42.545" y2="50.8" width="0.4064" layer="16"/>
+<wire x1="42.545" y1="50.8" x2="42.545" y2="61.595" width="0.4064" layer="16"/>
 </signal>
 <signal name="S$15">
 <contactref element="LD8" pad="AX"/>
 <contactref element="U1" pad="16"/>
-<wire x1="42.545" y1="46.355" x2="36.83" y2="46.355" width="0.4064" layer="16"/>
-<wire x1="36.83" y1="46.355" x2="36.83" y2="26.035" width="0.4064" layer="16"/>
+<wire x1="36.83" y1="26.035" x2="36.83" y2="34.29" width="0.4064" layer="16"/>
+<wire x1="36.83" y1="34.29" x2="42.545" y2="34.29" width="0.4064" layer="16"/>
+<wire x1="42.545" y1="34.29" x2="42.545" y2="46.355" width="0.4064" layer="16"/>
 </signal>
 <signal name="S$16">
@@
 <wire x1="39.37" y1="31.115" x2="42.545" y2="31.115" width="0.4064" layer="16"/>
 </signal>
+<signal name="S$19">
+<contactref element="U1" pad="11"/>
+<contactref element="JP3" pad="1"/>
+<wire x1="31.75" y1="18.415" x2="31.75" y2="21.59" width="0.4064" layer="16"/>
+<wire x1="31.75" y1="21.59" x2="35.56" y2="21.59" width="0.4064" layer="16"/>
+<wire x1="35.56" y1="21.59" x2="35.56" y2="36.83" width="0.4064" layer="16"/>
+<wire x1="35.56" y1="49.53" x2="35.56" y2="42.545" width="0.4064" layer="16"/>
+<wire x1="35.56" y1="42.545" x2="35.56" y2="36.83" width="0" layer="19" extent="1-16"/>
+</signal>
 </signals>

Commit message: tiny improvement (rotated LED)
Parts:
- turned LD9 to 270 degrees
Routing:
- net S$16: track 8.26 -> 13.3 mm
- net S$12: track 21.0 -> 15.9 mm
- net VCC: track 196.2 -> 200.0 mm
- net S$11: track 45.1 -> 43.8 mm
- net S$10: track 67.9 -> 66.7 mm
Other:
- board size 50.5 x 63.5 mm -> 49.8 x 63.5 mm
Changed lines of the file:
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@@
 <board>
 <plain>
-<wire x1="0.635" y1="1.905" x2="51.105" y2="1.905" width="0" layer="20"/>
-<wire x1="51.105" y1="1.905" x2="51.105" y2="65.395" width="0" layer="20"/>
-<wire x1="51.105" y1="65.395" x2="0.635" y2="65.395" width="0" layer="20"/>
+<wire x1="0.635" y1="1.905" x2="50.47" y2="1.905" width="0" layer="20"/>
+<wire x1="50.47" y1="1.905" x2="50.47" y2="65.395" width="0" layer="20"/>
+<wire x1="50.47" y1="65.395" x2="0.635" y2="65.395" width="0" layer="20"/>
 <wire x1="0.635" y1="65.395" x2="0.635" y2="1.905" width="0" layer="20"/>
 </plain>
@@
 <element name="LD7" library="led" package="DUOLED-C-5MM" value="" x="5.715" y="31.115"/>
 <element name="LD8" library="led" package="DUOLED-C-5MM" value="" x="45.085" y="46.355"/>
-<element name="LD9" library="led" package="DUOLED-C-5MM" value="" x="45.085" y="31.115"/>
+<element name="LD9" library="led" package="DUOLED-C-5MM" value="" x="45.085" y="31.115" rot="R270"/>
 <element name="IC1" library="micro-philips" package="DIL16" value="PCF8574P" x="15.875" y="40.64" rot="R90">
 <attribute name="OC_NEWARK" value="11N8515" x="34.925" y="64.77" size="1.778" layer="27" rot="R90" display="off"/>
@@
 <contactref element="LD9" pad="C"/>
 <contactref element="LD8" pad="C"/>
-<wire x1="45.085" y1="46.355" x2="45.085" y2="31.115" width="0.4064" layer="16"/>
 <contactref element="LD1" pad="C"/>
 <contactref element="LD3" pad="C"/>
@@
 <wire x1="24.13" y1="23.495" x2="21.59" y2="23.495" width="0.4064" layer="16"/>
 <wire x1="21.59" y1="23.495" x2="21.59" y2="18.415" width="0.4064" layer="16"/>
+<wire x1="45.085" y1="46.355" x2="45.085" y2="38.1" width="0.4064" layer="16"/>
+<wire x1="45.085" y1="38.1" x2="46.99" y2="38.1" width="0.4064" layer="16"/>
+<wire x1="46.99" y1="38.1" x2="46.99" y2="31.115" width="0.4064" layer="16"/>
+<wire x1="46.99" y1="31.115" x2="45.085" y2="31.115" width="0.4064" layer="16"/>
 </signal>
 <signal name="N$2">
@@
 <contactref element="LD3" pad="AR"/>
 <wire x1="34.29" y1="18.415" x2="34.29" y2="15.24" width="0.4064" layer="16"/>
-<wire x1="34.29" y1="15.24" x2="50.165" y2="15.24" width="0.4064" layer="16"/>
-<wire x1="50.165" y1="15.24" x2="50.165" y2="61.595" width="0.4064" layer="16"/>
-<wire x1="50.165" y1="61.595" x2="47.625" y2="61.595" width="0.4064" layer="16"/>
+<wire x1="34.29" y1="15.24" x2="49.53" y2="15.24" width="0.4064" layer="16"/>
+<wire x1="49.53" y1="15.24" x2="49.53" y2="61.595" width="0.4064" layer="16"/>
+<wire x1="49.53" y1="61.595" x2="47.625" y2="61.595" width="0.4064" layer="16"/>
 </signal>
 <signal name="S$11">
@@
 <contactref element="LD8" pad="AR"/>
 <wire x1="36.83" y1="18.415" x2="36.83" y2="16.51" width="0.4064" layer="16"/>
-<wire x1="36.83" y1="16.51" x2="48.895" y2="16.51" width="0.4064" layer="16"/>
-<wire x1="48.895" y1="16.51" x2="48.895" y2="46.355" width="0.4064" layer="16"/>
-<wire x1="48.895" y1="46.355" x2="47.625" y2="46.355" width="0.4064" layer="16"/>
+<wire x1="36.83" y1="16.51" x2="48.26" y2="16.51" width="0.4064" layer="16"/>
+<wire x1="48.26" y1="16.51" x2="48.26" y2="46.355" width="0.4064" layer="16"/>
+<wire x1="48.26" y1="46.355" x2="47.625" y2="46.355" width="0.4064" layer="16"/>
 </signal>
 <signal name="S$12">
 <contactref element="U1" pad="14"/>
 <contactref element="LD9" pad="AR"/>
-<wire x1="39.37" y1="18.415" x2="47.625" y2="18.415" width="0.4064" layer="16"/>
-<wire x1="47.625" y1="18.415" x2="47.625" y2="31.115" width="0.4064" layer="16"/>
+<wire x1="39.37" y1="18.415" x2="45.085" y2="18.415" width="0.4064" layer="16"/>
+<wire x1="45.085" y1="18.415" x2="45.085" y2="28.575" width="0.4064" layer="16"/>
 </signal>
 <signal name="S$6">
@@
 <contactref element="LD8" pad="AX"/>
 <contactref element="U1" pad="16"/>
-<wire x1="36.83" y1="26.035" x2="36.83" y2="34.29" width="0.4064" layer="16"/>
-<wire x1="36.83" y1="34.29" x2="42.545" y2="34.29" width="0.4064" layer="16"/>
-<wire x1="42.545" y1="34.29" x2="42.545" y2="46.355" width="0.4064" layer="16"/>
+<wire x1="36.83" y1="26.035" x2="36.83" y2="34.925" width="0.4064" layer="16"/>
+<wire x1="36.83" y1="34.925" x2="42.545" y2="34.925" width="0.4064" layer="16"/>
+<wire x1="42.545" y1="34.925" x2="42.545" y2="46.355" width="0.4064" layer="16"/>
 </signal>
 <signal name="S$16">
@@
 <wire x1="39.37" y1="26.035" x2="39.37" y2="31.115" width="0.4064" layer="16"/>
 <wire x1="39.37" y1="31.115" x2="42.545" y2="31.115" width="0.4064" layer="16"/>
+<wire x1="42.545" y1="31.115" x2="42.545" y2="33.655" width="0.4064" layer="16"/>
+<wire x1="42.545" y1="33.655" x2="45.085" y2="33.655" width="0.4064" layer="16"/>
 </signal>
 <signal name="S$19">

Commit message: fix: LED3 connection through JP3
Parts:
- moved JP3 1.91 mm to (37.5, 49.5)
Routing:
- net S$19: track 29.2 -> 36.8 mm
- net GND: track 170.9 -> 172.9 mm
- net S$14: track 42.7 -> 43.8 mm
Changed lines of the file:
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@@
 <element name="JP2" library="SparkFun-Connectors" package="1X03" value="" x="6.35" y="14.605"/>
 <element name="IC2" library="ic-package" package="SOCKET-08" value="" x="37.465" y="7.62" rot="R270"/>
-<element name="JP3" library="SparkFun-Connectors" package="1X04" value="" x="35.56" y="49.53" rot="R90"/>
+<element name="JP3" library="SparkFun-Connectors" package="1X04" value="" x="37.465" y="49.53" rot="R90"/>
 </elements>
 <signals>
@@
 <wire x1="28.2956" y1="10.2362" x2="27.94" y2="9.525" width="0.4064" layer="16"/>
 <wire x1="27.94" y1="9.525" x2="27.94" y2="8.255" width="0.4064" layer="16"/>
-<wire x1="35.56" y1="57.15" x2="33.02" y2="57.15" width="0.4064" layer="16"/>
+<wire x1="37.465" y1="57.15" x2="33.02" y2="57.15" width="0.4064" layer="16"/>
 <wire x1="33.02" y1="57.15" x2="33.02" y2="24.13" width="0.4064" layer="16"/>
 <wire x1="33.02" y1="24.13" x2="27.94" y2="24.13" width="0.4064" layer="16"/>
@@
 <contactref element="LD3" pad="AX"/>
 <contactref element="U1" pad="17"/>
-<wire x1="34.29" y1="26.035" x2="34.29" y2="39.37" width="0.4064" layer="16"/>
-<wire x1="34.29" y1="39.37" x2="40.64" y2="39.37" width="0.4064" layer="16"/>
-<wire x1="40.64" y1="39.37" x2="40.64" y2="48.895" width="0.4064" layer="16"/>
-<wire x1="40.64" y1="48.895" x2="42.545" y2="50.8" width="0.4064" layer="16"/>
-<wire x1="42.545" y1="50.8" x2="42.545" y2="61.595" width="0.4064" layer="16"/>
+<wire x1="34.29" y1="26.035" x2="34.29" y2="53.34" width="0.4064" layer="16"/>
+<wire x1="34.29" y1="53.34" x2="42.545" y2="53.34" width="0.4064" layer="16"/>
+<wire x1="42.545" y1="53.34" x2="42.545" y2="61.595" width="0.4064" layer="16"/>
 </signal>
 <signal name="S$15">
@@
 <wire x1="31.75" y1="21.59" x2="35.56" y2="21.59" width="0.4064" layer="16"/>
 <wire x1="35.56" y1="21.59" x2="35.56" y2="36.83" width="0.4064" layer="16"/>
-<wire x1="35.56" y1="49.53" x2="35.56" y2="42.545" width="0.4064" layer="16"/>
-<wire x1="35.56" y1="42.545" x2="35.56" y2="36.83" width="0" layer="19" extent="1-16"/>
+<wire x1="37.465" y1="49.53" x2="37.465" y2="36.83" width="0.4064" layer="16"/>
+<wire x1="37.465" y1="36.83" x2="35.56" y2="36.83" width="0.4064" layer="16"/>
 </signal>
 </signals>

Commit message: added 2nd ground and rotated LD4
Parts:
- turned LD4 to 270 degrees
Connections:
- net GND: now also U1.22
Routing:
- net S$8: track 17.1 -> 10.8 mm
- net VCC: track 200.0 -> 205.1 mm
- net GND: track 172.9 -> 174.8 mm
Changed lines of the file:
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@@
 <element name="LD2" library="led" package="DUOLED-C-5MM" value="" x="25.4" y="61.595"/>
 <element name="LD3" library="led" package="DUOLED-C-5MM" value="" x="45.085" y="61.595"/>
-<element name="LD4" library="led" package="DUOLED-C-5MM" value="" x="5.715" y="46.355"/>
+<element name="LD4" library="led" package="DUOLED-C-5MM" value="" x="5.715" y="46.355" rot="R270"/>
 <element name="LD5" library="led" package="DUOLED-C-5MM" value="" x="25.4" y="46.355"/>
 <element name="LD6" library="led" package="DUOLED-C-5MM" value="" x="25.4" y="31.115"/>
@@
 <wire x1="17.145" y1="29.845" x2="19.05" y2="29.845" width="0.4064" layer="16"/>
 <wire x1="19.05" y1="29.845" x2="19.05" y2="27.94" width="0.4064" layer="16"/>
-<wire x1="19.05" y1="27.94" x2="27.94" y2="27.94" width="0.4064" layer="16"/>
+<wire x1="19.05" y1="27.94" x2="21.59" y2="27.94" width="0.4064" layer="16"/>
+<wire x1="21.59" y1="27.94" x2="27.94" y2="27.94" width="0.4064" layer="16"/>
 <wire x1="27.94" y1="27.94" x2="27.94" y2="24.13" width="0.4064" layer="16"/>
 <contactref element="S3" pad="1"/>
@@
 <wire x1="33.02" y1="57.15" x2="33.02" y2="24.13" width="0.4064" layer="16"/>
 <wire x1="33.02" y1="24.13" x2="27.94" y2="24.13" width="0.4064" layer="16"/>
+<contactref element="U1" pad="22"/>
+<wire x1="21.59" y1="26.035" x2="21.59" y2="27.94" width="0.4064" layer="16"/>
 </signal>
 <signal name="VCC">
@@
 <wire x1="14.605" y1="31.75" x2="12.065" y2="31.75" width="0.4064" layer="16"/>
 <contactref element="LD7" pad="C"/>
-<wire x1="5.715" y1="31.115" x2="5.715" y2="38.1" width="0.4064" layer="16"/>
-<wire x1="5.715" y1="38.1" x2="14.605" y2="38.1" width="0.4064" layer="16"/>
+<wire x1="5.715" y1="31.115" x2="5.715" y2="37.465" width="0.4064" layer="16"/>
+<wire x1="5.715" y1="37.465" x2="14.605" y2="38.1" width="0.4064" layer="16"/>
 <wire x1="14.605" y1="38.1" x2="14.605" y2="31.75" width="0.4064" layer="16"/>
 <contactref element="LD4" pad="C"/>
-<wire x1="5.715" y1="46.355" x2="5.715" y2="38.1" width="0.4064" layer="16"/>
 <contactref element="LD9" pad="C"/>
 <contactref element="LD8" pad="C"/>
@@
 <wire x1="46.99" y1="38.1" x2="46.99" y2="31.115" width="0.4064" layer="16"/>
 <wire x1="46.99" y1="31.115" x2="45.085" y2="31.115" width="0.4064" layer="16"/>
+<wire x1="5.715" y1="37.465" x2="3.175" y2="37.465" width="0.4064" layer="16"/>
+<wire x1="3.175" y1="37.465" x2="3.175" y2="46.355" width="0.4064" layer="16"/>
+<wire x1="3.175" y1="46.355" x2="5.715" y2="46.355" width="0.4064" layer="16"/>
 </signal>
 <signal name="N$2">
@@
 <contactref element="LD4" pad="AR"/>
 <contactref element="IC1" pad="12"/>
-<wire x1="12.065" y1="41.91" x2="8.255" y2="41.91" width="0.4064" layer="16"/>
-<wire x1="8.255" y1="41.91" x2="8.255" y2="46.355" width="0.4064" layer="16"/>
+<wire x1="12.065" y1="41.91" x2="5.715" y2="41.91" width="0.4064" layer="16"/>
+<wire x1="5.715" y1="41.91" x2="5.715" y2="43.815" width="0.4064" layer="16"/>
 </signal>
 <signal name="S$8">
 <contactref element="LD4" pad="AX"/>
 <contactref element="IC1" pad="11"/>
-<wire x1="12.065" y1="44.45" x2="9.525" y2="44.45" width="0.4064" layer="16"/>
-<wire x1="9.525" y1="44.45" x2="9.525" y2="49.53" width="0.4064" layer="16"/>
-<wire x1="9.525" y1="49.53" x2="3.175" y2="49.53" width="0.4064" layer="16"/>
-<wire x1="3.175" y1="49.53" x2="3.175" y2="46.355" width="0.4064" layer="16"/>
+<wire x1="12.065" y1="44.45" x2="8.89" y2="44.45" width="0.4064" layer="16"/>
+<wire x1="8.89" y1="44.45" x2="8.89" y2="48.895" width="0.4064" layer="16"/>
+<wire x1="8.89" y1="48.895" x2="5.715" y2="48.895" width="0.4064" layer="16"/>
 </signal>
 <signal name="S$9">

Commit message: Piezo on VCC instead of ground (simplification)
Connections:
- net GND: no longer JP3.4
- net VCC: now also JP3.4
Routing:
- net GND: track 174.8 -> 132.2 mm
- net VCC: track 205.1 -> 212.7 mm
Changed lines of the file:
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@@
 <contactref element="IC2" pad="5"/>
 <contactref element="IC2" pad="3"/>
-<contactref element="JP3" pad="4"/>
 <wire x1="24.13" y1="18.415" x2="24.13" y2="14.605" width="0.4064" layer="16"/>
 <wire x1="24.13" y1="13.335" x2="24.13" y2="14.605" width="0.4064" layer="16"/>
@@
 <wire x1="28.2956" y1="10.2362" x2="27.94" y2="9.525" width="0.4064" layer="16"/>
 <wire x1="27.94" y1="9.525" x2="27.94" y2="8.255" width="0.4064" layer="16"/>
-<wire x1="37.465" y1="57.15" x2="33.02" y2="57.15" width="0.4064" layer="16"/>
-<wire x1="33.02" y1="57.15" x2="33.02" y2="24.13" width="0.4064" layer="16"/>
-<wire x1="33.02" y1="24.13" x2="27.94" y2="24.13" width="0.4064" layer="16"/>
 <contactref element="U1" pad="22"/>
 <wire x1="21.59" y1="26.035" x2="21.59" y2="27.94" width="0.4064" layer="16"/>
@@
 <contactref element="LD1" pad="C"/>
 <contactref element="LD3" pad="C"/>
-<wire x1="45.085" y1="61.595" x2="45.085" y2="46.355" width="0.4064" layer="16"/>
+<wire x1="45.085" y1="61.595" x2="45.085" y2="57.15" width="0.4064" layer="16"/>
+<wire x1="45.085" y1="57.15" x2="45.085" y2="46.355" width="0.4064" layer="16"/>
 <wire x1="45.085" y1="63.5" x2="45.085" y2="61.595" width="0.4064" layer="16"/>
 <wire x1="5.715" y1="63.5" x2="5.715" y2="61.595" width="0.4064" layer="16"/>
@@
 <wire x1="3.175" y1="37.465" x2="3.175" y2="46.355" width="0.4064" layer="16"/>
 <wire x1="3.175" y1="46.355" x2="5.715" y2="46.355" width="0.4064" layer="16"/>
+<contactref element="JP3" pad="4"/>
+<wire x1="37.465" y1="57.15" x2="45.085" y2="57.15" width="0.4064" layer="16"/>
 </signal>
 <signal name="N$2">
@@
 <contactref element="LD3" pad="AX"/>
 <contactref element="U1" pad="17"/>
-<wire x1="34.29" y1="26.035" x2="34.29" y2="53.34" width="0.4064" layer="16"/>
-<wire x1="34.29" y1="53.34" x2="42.545" y2="53.34" width="0.4064" layer="16"/>
-<wire x1="42.545" y1="53.34" x2="42.545" y2="61.595" width="0.4064" layer="16"/>
+<wire x1="34.29" y1="26.035" x2="34.29" y2="61.595" width="0.4064" layer="16"/>
+<wire x1="34.29" y1="61.595" x2="42.545" y2="61.595" width="0.4064" layer="16"/>
 </signal>
 <signal name="S$15">

Commit message: tiny fixes
Parts:
- moved IC2 3.86 mm to (41.3, 8.26)
Connections:
- net S$11: now also JP3.1, U1.16; no longer LD8.AR, U1.13
- net S$12: now also LD8.AX, U1.15; no longer LD9.AR, U1.14
- net S$15: now also LD8.AR, U1.13; no longer LD8.AX, U1.16
- net S$16: now also LD9.AR, U1.14; no longer LD9.AX, U1.15
- net S$19: now also LD9.AX; no longer JP3.1
Routing:
- net S$11: track 43.8 -> 24.1 mm
- net S$15: track 26.0 -> 43.8 mm
- net VCC: track 212.7 -> 230.5 mm
- net S$19: track 36.8 -> 28.6 mm
- net S$12: track 15.9 -> 23.5 mm
- net N$8: track 23.5 -> 27.3 mm
- net N$7: track 26.7 -> 29.8 mm
- net S$16: track 13.3 -> 15.9 mm
- net GND: track 132.2 -> 134.6 mm
