File: Donjan/tictactoe2.brd (EAGLE design)
At the start: 49.8 x 63.5 mm, 18 parts, among them IC1 PCF8574P, U1 ATMEGA328P_PDIP

Commit message: tiny fixes #3
Parts:
- moved JP3 1.91 mm to (35.6, 49.5)
Routing:
- net S$14: track 43.8 -> 46.4 mm
- net VCC: track 230.5 -> 232.4 mm
- net S$11: track 24.1 -> 24.8 mm
Changed lines of the file:
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@@
 <element name="JP2" library="SparkFun-Connectors" package="1X03" value="" x="6.35" y="14.605"/>
 <element name="IC2" library="ic-package" package="SOCKET-08" value="" x="41.275" y="8.255" rot="R270"/>
-<element name="JP3" library="SparkFun-Connectors" package="1X04" value="" x="37.465" y="49.53" rot="R90"/>
+<element name="JP3" library="SparkFun-Connectors" package="1X04" value="" x="35.56" y="49.53" rot="R90"/>
 </elements>
 <signals>
@@
 <wire x1="1.905" y1="46.355" x2="5.715" y2="46.355" width="0.4064" layer="16"/>
 <contactref element="JP3" pad="4"/>
-<wire x1="37.465" y1="57.15" x2="45.085" y2="57.15" width="0.4064" layer="16"/>
+<wire x1="35.56" y1="57.15" x2="45.085" y2="57.15" width="0.4064" layer="16"/>
 <wire x1="5.715" y1="37.465" x2="1.905" y2="37.465" width="0.4064" layer="16"/>
 <wire x1="1.905" y1="37.465" x2="1.905" y2="46.355" width="0.4064" layer="16"/>
@@
 <contactref element="LD3" pad="AX"/>
 <contactref element="U1" pad="17"/>
-<wire x1="34.29" y1="26.035" x2="34.29" y2="61.595" width="0.4064" layer="16"/>
-<wire x1="34.29" y1="61.595" x2="42.545" y2="61.595" width="0.4064" layer="16"/>
+<wire x1="33.02" y1="61.595" x2="42.545" y2="61.595" width="0.4064" layer="16"/>
+<wire x1="34.29" y1="26.035" x2="34.29" y2="28.575" width="0.4064" layer="16"/>
+<wire x1="34.29" y1="28.575" x2="33.02" y2="28.575" width="0.4064" layer="16"/>
+<wire x1="33.02" y1="28.575" x2="33.02" y2="61.595" width="0.4064" layer="16"/>
 </signal>
 <signal name="S$11">
@@
 <contactref element="JP3" pad="1"/>
 <wire x1="36.83" y1="26.035" x2="36.83" y2="49.53" width="0.4064" layer="16"/>
-<wire x1="36.83" y1="49.53" x2="37.465" y2="49.53" width="0.4064" layer="16"/>
+<wire x1="36.83" y1="49.53" x2="35.56" y2="49.53" width="0.4064" layer="16"/>
 </signal>
 <signal name="S$12">
