File: Cyrill/clock_one/watch_one.sch (EAGLE design)
At the start: 22 parts, among them U1 ATMEGA328P_PDIP

Commit message: clock_try2
Parts:
- removed IC1: (no value), ic-package:DIL8S
- added SL1, SL2: (no value), con-amp-quick:M02
- added Y1: (no value), SparkFun-FreqCtrl:CRYSTALHC49US
- JP5, JP7, JP8, JP9: value M01PTH_2MM -> M01SMD; device SparkFun-Connectors:M01PTH_2MM -> SparkFun-Connectors:M01SMD
Connections:
- net GND: now also SL1.1, SL2.1; no longer IC1.3, IC1.5
- net N$19: now also SL1.2, Y1.1; no longer IC1.1, IC1.4
- net N$20: now also SL2.2, Y1.2; no longer IC1.6, IC1.8
Changed lines of the file:
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@@
 <part name="LED10" library="SparkFun-LED" deviceset="LED" device="3MM"/>
 <part name="LED11" library="SparkFun-LED" deviceset="LED" device="3MM"/>
-<part name="JP5" library="SparkFun-Connectors" deviceset="M01" device="PTH_2MM"/>
-<part name="JP7" library="SparkFun-Connectors" deviceset="M01" device="PTH_2MM"/>
-<part name="JP8" library="SparkFun-Connectors" deviceset="M01" device="PTH_2MM"/>
-<part name="JP9" library="SparkFun-Connectors" deviceset="M01" device="PTH_2MM"/>
-<part name="IC1" library="ic-package" deviceset="DIL8" device="S"/>
+<part name="JP5" library="SparkFun-Connectors" deviceset="M01" device="SMD" value="M01SMD"/>
+<part name="JP7" library="SparkFun-Connectors" deviceset="M01" device="SMD" value="M01SMD"/>
+<part name="JP8" library="SparkFun-Connectors" deviceset="M01" device="SMD" value="M01SMD"/>
+<part name="JP9" library="SparkFun-Connectors" deviceset="M01" device="SMD" value="M01SMD"/>
+<part name="Y1" library="SparkFun-FreqCtrl" deviceset="CRYSTAL" device="HC49US"/>
+<part name="SL1" library="con-amp-quick" deviceset="M02" device=""/>
+<part name="SL2" library="con-amp-quick" deviceset="M02" device=""/>
 </parts>
 <sheets>
@@
 <instance part="JP8" gate="G$1" x="68.58" y="-22.86"/>
 <instance part="JP9" gate="G$1" x="48.26" y="-22.86"/>
-<instance part="IC1" gate="G$1" x="10.16" y="27.94"/>
+<instance part="Y1" gate="G$1" x="10.16" y="12.7"/>
+<instance part="SL1" gate="G$1" x="10.16" y="0"/>
+<instance part="SL2" gate="G$1" x="10.16" y="-12.7"/>
 </instances>
 <busses>
@@
 <wire x1="15.24" y1="43.18" x2="25.4" y2="43.18" width="0.1524" layer="91"/>
 <wire x1="25.4" y1="43.18" x2="25.4" y2="17.78" width="0.1524" layer="91"/>
-<wire x1="25.4" y1="17.78" x2="33.02" y2="17.78" width="0.1524" layer="91"/>
+<wire x1="25.4" y1="17.78" x2="30.48" y2="17.78" width="0.1524" layer="91"/>
+<wire x1="30.48" y1="17.78" x2="33.02" y2="17.78" width="0.1524" layer="91"/>
 <wire x1="33.02" y1="17.78" x2="38.1" y2="17.78" width="0.1524" layer="91"/>
 <wire x1="55.88" y1="2.54" x2="25.4" y2="2.54" width="0.1524" layer="91"/>
@@
 <wire x1="-2.54" y1="104.14" x2="-2.54" y2="17.78" width="0.1524" layer="91"/>
 <wire x1="-2.54" y1="17.78" x2="25.4" y2="17.78" width="0.1524" layer="91"/>
-<pinref part="IC1" gate="G$1" pin="3"/>
 <wire x1="2.54" y1="25.4" x2="10.16" y2="25.4" width="0.1524" layer="91"/>
 <wire x1="10.16" y1="25.4" x2="10.16" y2="22.86" width="0.1524" layer="91"/>
-<pinref part="IC1" gate="G$1" pin="5"/>
-<wire x1="10.16" y1="22.86" x2="17.78" y2="22.86" width="0.1524" layer="91"/>
-<wire x1="17.78" y1="22.86" x2="33.02" y2="22.86" width="0.1524" layer="91"/>
+<wire x1="10.16" y1="22.86" x2="33.02" y2="22.86" width="0.1524" layer="91"/>
 <wire x1="33.02" y1="22.86" x2="33.02" y2="17.78" width="0.1524" layer="91"/>
-<junction x="17.78" y="22.86"/>
 <junction x="33.02" y="17.78"/>
+<pinref part="SL1" gate="G$1" pin="1"/>
+<wire x1="17.78" y1="0" x2="20.32" y2="0" width="0.1524" layer="91"/>
+<wire x1="20.32" y1="0" x2="20.32" y2="-2.54" width="0.1524" layer="91"/>
+<wire x1="20.32" y1="-2.54" x2="30.48" y2="-2.54" width="0.1524" layer="91"/>
+<wire x1="30.48" y1="-2.54" x2="30.48" y2="17.78" width="0.1524" layer="91"/>
+<junction x="30.48" y="17.78"/>
+<pinref part="SL2" gate="G$1" pin="1"/>
+<wire x1="17.78" y1="-12.7" x2="20.32" y2="-12.7" width="0.1524" layer="91"/>
+<wire x1="20.32" y1="-12.7" x2="20.32" y2="-20.32" width="0.1524" layer="91"/>
+<wire x1="20.32" y1="-20.32" x2="-2.54" y2="-20.32" width="0.1524" layer="91"/>
+<wire x1="-2.54" y1="-20.32" x2="-2.54" y2="17.78" width="0.1524" layer="91"/>
+<junction x="-2.54" y="17.78"/>
 </segment>
 </net>
@@
 <net name="N$19" class="0">
 <segment>
-<pinref part="IC1" gate="G$1" pin="1"/>
-<wire x1="2.54" y1="30.48" x2="0" y2="30.48" width="0.1524" layer="91"/>
-<wire x1="0" y1="30.48" x2="0" y2="35.56" width="0.1524" layer="91"/>
 <wire x1="0" y1="35.56" x2="33.02" y2="35.56" width="0.1524" layer="91"/>
 <wire x1="33.02" y1="35.56" x2="33.02" y2="45.72" width="0.1524" layer="91"/>
 <wire x1="33.02" y1="45.72" x2="38.1" y2="45.72" width="0.1524" layer="91"/>
 <wire x1="38.1" y1="45.72" x2="40.64" y2="45.72" width="0.1524" layer="91"/>
-<wire x1="0" y1="30.48" x2="0" y2="22.86" width="0.1524" layer="91"/>
-<junction x="0" y="30.48"/>
-<pinref part="IC1" gate="G$1" pin="4"/>
+<wire x1="0" y1="35.56" x2="0" y2="22.86" width="0.1524" layer="91"/>
 <wire x1="0" y1="22.86" x2="2.54" y2="22.86" width="0.1524" layer="91"/>
 <pinref part="U1" gate="G$1" pin="PB6(XTAL1/TOSC1)"/>
 <junction x="38.1" y="45.72"/>
+<wire x1="0" y1="22.86" x2="0" y2="12.7" width="0.1524" layer="91"/>
+<junction x="0" y="22.86"/>
+<pinref part="Y1" gate="G$1" pin="1"/>
+<wire x1="0" y1="12.7" x2="7.62" y2="12.7" width="0.1524" layer="91"/>
+<pinref part="SL1" gate="G$1" pin="2"/>
+<wire x1="17.78" y1="2.54" x2="17.78" y2="7.62" width="0.1524" layer="91"/>
+<wire x1="17.78" y1="7.62" x2="0" y2="7.62" width="0.1524" layer="91"/>
+<wire x1="0" y1="7.62" x2="0" y2="12.7" width="0.1524" layer="91"/>
+<junction x="0" y="12.7"/>
 </segment>
 </net>
 <net name="N$20" class="0">
 <segment>
-<pinref part="IC1" gate="G$1" pin="8"/>
 <pinref part="U1" gate="G$1" pin="PB7(XTAL2/TOSC2)"/>
-<wire x1="17.78" y1="30.48" x2="27.94" y2="30.48" width="0.1524" layer="91"/>
-<wire x1="27.94" y1="30.48" x2="38.1" y2="30.48" width="0.1524" layer="91"/>
+<wire x1="27.94" y1="30.48" x2="35.56" y2="30.48" width="0.1524" layer="91"/>
+<wire x1="35.56" y1="30.48" x2="38.1" y2="30.48" width="0.1524" layer="91"/>
 <wire x1="38.1" y1="30.48" x2="38.1" y2="40.64" width="0.1524" layer="91"/>
-<pinref part="IC1" gate="G$1" pin="6"/>
 <wire x1="17.78" y1="25.4" x2="27.94" y2="25.4" width="0.1524" layer="91"/>
 <wire x1="27.94" y1="25.4" x2="27.94" y2="30.48" width="0.1524" layer="91"/>
+<pinref part="Y1" gate="G$1" pin="2"/>
+<wire x1="12.7" y1="12.7" x2="20.32" y2="12.7" width="0.1524" layer="91"/>
+<wire x1="20.32" y1="12.7" x2="20.32" y2="30.48" width="0.1524" layer="91"/>
+<wire x1="20.32" y1="30.48" x2="27.94" y2="30.48" width="0.1524" layer="91"/>
 <junction x="27.94" y="30.48"/>
-</segment>
-</net>
+<pinref part="SL2" gate="G$1" pin="2"/>
+<wire x1="17.78" y1="-10.16" x2="35.56" y2="-10.16" width="0.1524" layer="91"/>
+<wire x1="35.56" y1="-10.16" x2="35.56" y2="30.48" width="0.1524" layer="91"/>
+<junction x="35.56" y="30.48"/>
+</segment>
+</net>

Commit message: clock_one minor adjustments pcb
Changed lines of the file:
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@@
 <wire x1="25.4" y1="43.18" x2="25.4" y2="17.78" width="0.1524" layer="91"/>
 <wire x1="25.4" y1="17.78" x2="30.48" y2="17.78" width="0.1524" layer="91"/>
-<wire x1="30.48" y1="17.78" x2="33.02" y2="17.78" width="0.1524" layer="91"/>
-<wire x1="33.02" y1="17.78" x2="38.1" y2="17.78" width="0.1524" layer="91"/>
+<wire x1="30.48" y1="17.78" x2="38.1" y2="17.78" width="0.1524" layer="91"/>
 <wire x1="55.88" y1="2.54" x2="25.4" y2="2.54" width="0.1524" layer="91"/>
 <wire x1="25.4" y1="2.54" x2="25.4" y2="17.78" width="0.1524" layer="91"/>
@@
 <wire x1="-2.54" y1="104.14" x2="-2.54" y2="17.78" width="0.1524" layer="91"/>
 <wire x1="-2.54" y1="17.78" x2="25.4" y2="17.78" width="0.1524" layer="91"/>
-<wire x1="2.54" y1="25.4" x2="10.16" y2="25.4" width="0.1524" layer="91"/>
-<wire x1="10.16" y1="25.4" x2="10.16" y2="22.86" width="0.1524" layer="91"/>
-<wire x1="10.16" y1="22.86" x2="33.02" y2="22.86" width="0.1524" layer="91"/>
-<wire x1="33.02" y1="22.86" x2="33.02" y2="17.78" width="0.1524" layer="91"/>
-<junction x="33.02" y="17.78"/>
 <pinref part="SL1" gate="G$1" pin="1"/>
 <wire x1="17.78" y1="0" x2="20.32" y2="0" width="0.1524" layer="91"/>
@@
 <wire x1="33.02" y1="45.72" x2="38.1" y2="45.72" width="0.1524" layer="91"/>
 <wire x1="38.1" y1="45.72" x2="40.64" y2="45.72" width="0.1524" layer="91"/>
-<wire x1="0" y1="35.56" x2="0" y2="22.86" width="0.1524" layer="91"/>
-<wire x1="0" y1="22.86" x2="2.54" y2="22.86" width="0.1524" layer="91"/>
+<wire x1="0" y1="35.56" x2="0" y2="12.7" width="0.1524" layer="91"/>
 <pinref part="U1" gate="G$1" pin="PB6(XTAL1/TOSC1)"/>
 <junction x="38.1" y="45.72"/>
-<wire x1="0" y1="22.86" x2="0" y2="12.7" width="0.1524" layer="91"/>
-<junction x="0" y="22.86"/>
 <pinref part="Y1" gate="G$1" pin="1"/>
 <wire x1="0" y1="12.7" x2="7.62" y2="12.7" width="0.1524" layer="91"/>
@@
 <segment>
 <pinref part="U1" gate="G$1" pin="PB7(XTAL2/TOSC2)"/>
-<wire x1="27.94" y1="30.48" x2="35.56" y2="30.48" width="0.1524" layer="91"/>
 <wire x1="35.56" y1="30.48" x2="38.1" y2="30.48" width="0.1524" layer="91"/>
 <wire x1="38.1" y1="30.48" x2="38.1" y2="40.64" width="0.1524" layer="91"/>
-<wire x1="17.78" y1="25.4" x2="27.94" y2="25.4" width="0.1524" layer="91"/>
-<wire x1="27.94" y1="25.4" x2="27.94" y2="30.48" width="0.1524" layer="91"/>
 <pinref part="Y1" gate="G$1" pin="2"/>
 <wire x1="12.7" y1="12.7" x2="20.32" y2="12.7" width="0.1524" layer="91"/>
 <wire x1="20.32" y1="12.7" x2="20.32" y2="30.48" width="0.1524" layer="91"/>
-<wire x1="20.32" y1="30.48" x2="27.94" y2="30.48" width="0.1524" layer="91"/>
-<junction x="27.94" y="30.48"/>
+<wire x1="20.32" y1="30.48" x2="35.56" y2="30.48" width="0.1524" layer="91"/>
 <pinref part="SL2" gate="G$1" pin="2"/>
 <wire x1="17.78" y1="-10.16" x2="35.56" y2="-10.16" width="0.1524" layer="91"/>

Commit message: OUTLINE TOP BOTTOM DRILL tilt sensor to A0 correction
Connections:
- removed net N$6: JP4.2, U1.PD2(INT0)
- new net N$22: JP4.2, U1.PC0(ADC0)
- net N$18: now also U1.PD2(INT0); no longer U1.PC0(ADC0)
Changed lines of the file:
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@@
-</segment>
-</net>
-<net name="N$6" class="0">
-<segment>
-<pinref part="U1" gate="G$1" pin="PD2(INT0)"/>
-<wire x1="101.6" y1="96.52" x2="101.6" y2="43.18" width="0.1524" layer="91"/>
-<wire x1="101.6" y1="43.18" x2="86.36" y2="43.18" width="0.1524" layer="91"/>
-<pinref part="JP4" gate="G$1" pin="2"/>
-<wire x1="78.74" y1="96.52" x2="101.6" y2="96.52" width="0.1524" layer="91"/>
 </segment>
 </net>
@@
 <pinref part="JP6" gate="G$1" pin="3"/>
 <wire x1="40.64" y1="96.52" x2="53.34" y2="96.52" width="0.1524" layer="91"/>
-<wire x1="88.9" y1="106.68" x2="88.9" y2="71.12" width="0.1524" layer="91"/>
-<pinref part="U1" gate="G$1" pin="PC0(ADC0)"/>
-<wire x1="88.9" y1="71.12" x2="86.36" y2="71.12" width="0.1524" layer="91"/>
-<wire x1="53.34" y1="106.68" x2="88.9" y2="106.68" width="0.1524" layer="91"/>
+<wire x1="53.34" y1="106.68" x2="101.6" y2="106.68" width="0.1524" layer="91"/>
+<pinref part="U1" gate="G$1" pin="PD2(INT0)"/>
+<wire x1="101.6" y1="43.18" x2="86.36" y2="43.18" width="0.1524" layer="91"/>
+<wire x1="101.6" y1="106.68" x2="101.6" y2="43.18" width="0.1524" layer="91"/>
 </segment>
 </net>
@@
 </segment>
 </net>
+<net name="N$22" class="0">
+<segment>
+<pinref part="U1" gate="G$1" pin="PC0(ADC0)"/>
+<wire x1="88.9" y1="71.12" x2="86.36" y2="71.12" width="0.1524" layer="91"/>
+<pinref part="JP4" gate="G$1" pin="2"/>
+<wire x1="78.74" y1="96.52" x2="88.9" y2="96.52" width="0.1524" layer="91"/>
+<wire x1="88.9" y1="71.12" x2="88.9" y2="96.52" width="0.1524" layer="91"/>
+</segment>
+</net>

Commit message: schaltplan update
Connections:
- removed net N$15: LED11.C, U1.PD3(INT1)
- removed net N$17: JP3.2, U1.PC1(ADC1)
- new net SWAP1: JP3.2, U1.PD3(INT1)
- new net SWAP2: LED11.C, U1.PC1(ADC1)
- net VCC: now also U1.AVCC
Changed lines of the file:
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@@
 <wire x1="121.92" y1="93.98" x2="114.3" y2="93.98" width="0.1524" layer="91"/>
 <pinref part="JP1" gate="G$1" pin="2"/>
+<pinref part="U1" gate="G$1" pin="AVCC"/>
+<wire x1="38.1" y1="66.04" x2="38.1" y2="63.5" width="0.1524" layer="91"/>
+<junction x="38.1" y="63.5"/>
 </segment>
 </net>
@@
 </segment>
 </net>
-<net name="N$15" class="0">
+<net name="SWAP2" class="0">
 <segment>
 <pinref part="LED11" gate="G$1" pin="C"/>
 <wire x1="121.92" y1="-7.62" x2="101.6" y2="-7.62" width="0.1524" layer="91"/>
 <wire x1="101.6" y1="-7.62" x2="101.6" y2="40.64" width="0.1524" layer="91"/>
-<pinref part="U1" gate="G$1" pin="PD3(INT1)"/>
-<wire x1="101.6" y1="40.64" x2="86.36" y2="40.64" width="0.1524" layer="91"/>
+<wire x1="101.6" y1="40.64" x2="104.14" y2="40.64" width="0.1524" layer="91"/>
+<wire x1="104.14" y1="40.64" x2="104.14" y2="68.58" width="0.1524" layer="91"/>
+<pinref part="U1" gate="G$1" pin="PC1(ADC1)"/>
+<wire x1="104.14" y1="68.58" x2="86.36" y2="68.58" width="0.1524" layer="91"/>
 </segment>
 </net>
-<net name="N$17" class="0">
+<net name="SWAP1" class="0">
 <segment>
 <pinref part="JP3" gate="G$1" pin="2"/>
 <wire x1="114.3" y1="96.52" x2="114.3" y2="101.6" width="0.1524" layer="91"/>
 <wire x1="114.3" y1="101.6" x2="99.06" y2="101.6" width="0.1524" layer="91"/>
-<wire x1="99.06" y1="101.6" x2="99.06" y2="68.58" width="0.1524" layer="91"/>
-<pinref part="U1" gate="G$1" pin="PC1(ADC1)"/>
-<wire x1="99.06" y1="68.58" x2="86.36" y2="68.58" width="0.1524" layer="91"/>
+<wire x1="99.06" y1="101.6" x2="99.06" y2="40.64" width="0.1524" layer="91"/>
+<pinref part="U1" gate="G$1" pin="PD3(INT1)"/>
+<wire x1="99.06" y1="40.64" x2="86.36" y2="40.64" width="0.1524" layer="91"/>
 </segment>
 </net>
