File: Cyrill/clock_one/watch_one.brd (EAGLE design)
At the start: 105.4 x 41.9 mm, 24 parts, among them U1 ATMEGA328P_PDIP

Commit message: schaltplan next
Routing:
- net GND: track 167.6 -> 204.5 mm
Other:
- board size 105.4 x 41.9 mm -> 101.6 x 41.9 mm
Changed lines of the file:
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@@
 <wire x1="54.61" y1="53.34" x2="63.5" y2="53.34" width="0.4064" layer="20"/>
 <wire x1="63.5" y1="53.34" x2="63.5" y2="49.53" width="0.4064" layer="20"/>
-<wire x1="63.5" y1="49.53" x2="104.14" y2="49.53" width="0.4064" layer="20"/>
-<wire x1="104.14" y1="49.53" x2="104.14" y2="29.21" width="0.4064" layer="20"/>
-<wire x1="104.14" y1="29.21" x2="64.77" y2="29.21" width="0.4064" layer="20"/>
+<wire x1="63.5" y1="49.53" x2="100.33" y2="49.53" width="0.4064" layer="20"/>
+<wire x1="100.33" y1="49.53" x2="100.33" y2="29.21" width="0.4064" layer="20"/>
+<wire x1="100.33" y1="29.21" x2="64.77" y2="29.21" width="0.4064" layer="20"/>
 <wire x1="64.77" y1="29.21" x2="64.77" y2="25.4" width="0.4064" layer="20"/>
 <wire x1="64.77" y1="25.4" x2="54.61" y2="25.4" width="0.4064" layer="20"/>
@@
 <wire x1="52.07" y1="30.48" x2="78.74" y2="30.48" width="0.4064" layer="1"/>
 <wire x1="78.74" y1="30.48" x2="78.74" y2="33.02" width="0.4064" layer="1"/>
-<wire x1="6.35" y1="38.1" x2="5.08" y2="38.1" width="0.4064" layer="1"/>
-<wire x1="5.08" y1="38.1" x2="5.08" y2="27.94" width="0.4064" layer="1"/>
+<wire x1="19.05" y1="40.64" x2="33.02" y2="40.64" width="0.4064" layer="1"/>
+<wire x1="33.02" y1="40.64" x2="33.02" y2="25.4" width="0.4064" layer="1"/>
+<wire x1="33.02" y1="25.4" x2="52.07" y2="25.4" width="0.4064" layer="1"/>
 </signal>
 <signal name="VCC">
@@
 <wire x1="49.53" y1="30.48" x2="59.69" y2="30.48" width="0.4064" layer="16"/>
 <wire x1="59.69" y1="30.48" x2="59.69" y2="35.56" width="0.4064" layer="16"/>
-<wire x1="59.69" y1="35.56" x2="63.5" y2="35.56" width="0.4064" layer="16"/>
-<wire x1="63.5" y1="35.56" x2="63.5" y2="38.1" width="0.4064" layer="16"/>
-<wire x1="63.5" y1="38.1" x2="66.04" y2="38.1" width="0.4064" layer="16"/>
+<wire x1="59.69" y1="35.56" x2="66.04" y2="35.56" width="0.4064" layer="16"/>
+<wire x1="66.04" y1="35.56" x2="66.04" y2="38.1" width="0.4064" layer="16"/>
 </signal>
 <signal name="N$10">
@@
 <wire x1="13.97" y1="19.05" x2="53.34" y2="19.05" width="0.4064" layer="16"/>
 <wire x1="53.34" y1="19.05" x2="53.34" y2="26.67" width="0.4064" layer="16"/>
-<wire x1="63.5" y1="31.75" x2="67.31" y2="31.75" width="0.4064" layer="16"/>
-<wire x1="67.31" y1="31.75" x2="67.31" y2="33.02" width="0.4064" layer="16"/>
-<wire x1="67.31" y1="33.02" x2="71.12" y2="33.02" width="0.4064" layer="16"/>
-<wire x1="71.12" y1="33.02" x2="71.12" y2="34.29" width="0.4064" layer="16"/>
-<wire x1="71.12" y1="34.29" x2="74.93" y2="34.29" width="0.4064" layer="16"/>
-<wire x1="74.93" y1="34.29" x2="74.93" y2="35.56" width="0.4064" layer="16"/>
-<wire x1="74.93" y1="35.56" x2="78.74" y2="35.56" width="0.4064" layer="16"/>
+<wire x1="63.5" y1="31.75" x2="73.66" y2="31.75" width="0.4064" layer="16"/>
+<wire x1="73.66" y1="31.75" x2="73.66" y2="35.56" width="0.4064" layer="16"/>
+<wire x1="73.66" y1="35.56" x2="78.74" y2="35.56" width="0.4064" layer="16"/>
 <wire x1="78.74" y1="35.56" x2="78.74" y2="38.1" width="0.4064" layer="16"/>
 <wire x1="78.74" y1="38.1" x2="81.28" y2="38.1" width="0.4064" layer="16"/>
@@
 <wire x1="15.24" y1="25.4" x2="15.24" y2="20.32" width="0.4064" layer="16"/>
 <wire x1="15.24" y1="20.32" x2="52.07" y2="20.32" width="0.4064" layer="16"/>
-<wire x1="62.23" y1="33.02" x2="66.04" y2="33.02" width="0.4064" layer="16"/>
-<wire x1="66.04" y1="33.02" x2="66.04" y2="34.29" width="0.4064" layer="16"/>
-<wire x1="66.04" y1="34.29" x2="69.85" y2="34.29" width="0.4064" layer="16"/>
-<wire x1="69.85" y1="34.29" x2="69.85" y2="35.56" width="0.4064" layer="16"/>
-<wire x1="69.85" y1="35.56" x2="73.66" y2="35.56" width="0.4064" layer="16"/>
-<wire x1="73.66" y1="35.56" x2="73.66" y2="38.1" width="0.4064" layer="16"/>
-<wire x1="73.66" y1="38.1" x2="76.2" y2="38.1" width="0.4064" layer="16"/>
+<wire x1="62.23" y1="33.02" x2="72.39" y2="33.02" width="0.4064" layer="16"/>
+<wire x1="72.39" y1="33.02" x2="72.39" y2="36.83" width="0.4064" layer="16"/>
+<wire x1="72.39" y1="36.83" x2="76.2" y2="36.83" width="0.4064" layer="16"/>
+<wire x1="76.2" y1="36.83" x2="76.2" y2="38.1" width="0.4064" layer="16"/>
 <wire x1="62.23" y1="27.94" x2="52.07" y2="27.94" width="0.4064" layer="16"/>
 <wire x1="52.07" y1="27.94" x2="52.07" y2="20.32" width="0.4064" layer="16"/>
@@
 <wire x1="16.51" y1="25.4" x2="16.51" y2="21.59" width="0.4064" layer="16"/>
 <wire x1="16.51" y1="21.59" x2="50.8" y2="21.59" width="0.4064" layer="16"/>
-<wire x1="60.96" y1="34.29" x2="64.77" y2="34.29" width="0.4064" layer="16"/>
-<wire x1="64.77" y1="34.29" x2="64.77" y2="35.56" width="0.4064" layer="16"/>
-<wire x1="64.77" y1="35.56" x2="68.58" y2="35.56" width="0.4064" layer="16"/>
-<wire x1="68.58" y1="35.56" x2="68.58" y2="38.1" width="0.4064" layer="16"/>
-<wire x1="68.58" y1="38.1" x2="71.12" y2="38.1" width="0.4064" layer="16"/>
+<wire x1="60.96" y1="34.29" x2="71.12" y2="34.29" width="0.4064" layer="16"/>
+<wire x1="71.12" y1="34.29" x2="71.12" y2="38.1" width="0.4064" layer="16"/>
 <wire x1="60.96" y1="29.21" x2="50.8" y2="29.21" width="0.4064" layer="16"/>
 <wire x1="50.8" y1="29.21" x2="50.8" y2="21.59" width="0.4064" layer="16"/>
@@
 <vertex x="63.5" y="53.34"/>
 <vertex x="63.5" y="49.53"/>
-<vertex x="104.14" y="49.53"/>
-<vertex x="104.14" y="29.21"/>
+<vertex x="100.33" y="49.53"/>
+<vertex x="100.33" y="29.21"/>
 <vertex x="64.77" y="29.21"/>
 <vertex x="64.77" y="25.4"/>
@@
 <vertex x="63.5" y="53.34"/>
 <vertex x="63.5" y="49.53"/>
-<vertex x="104.14" y="49.53"/>
-<vertex x="104.14" y="29.21"/>
+<vertex x="100.33" y="49.53"/>
+<vertex x="100.33" y="29.21"/>
 <vertex x="64.77" y="29.21"/>
 <vertex x="64.77" y="25.4"/>
