File: Cyrill/clock_one/watch_one.brd (EAGLE design)
At the start: 101.6 x 41.9 mm, 24 parts, among them U1 ATMEGA328P_PDIP

Commit message: TOP BOTTOM OUTLINE DRILL next
Routing:
- net N$1: track 33.0 -> 31.7 mm
Other:
- outline, holes or cut-outs redrawn
Changed lines of the file:
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@@
 <wire x1="-1.27" y1="59.68" x2="-1.27" y2="17.78" width="0" layer="20"/>
 <wire x1="-1.27" y1="59.69" x2="54.61" y2="59.69" width="0.4064" layer="20"/>
-<wire x1="54.61" y1="59.69" x2="54.61" y2="53.34" width="0.4064" layer="20"/>
-<wire x1="54.61" y1="53.34" x2="63.5" y2="53.34" width="0.4064" layer="20"/>
-<wire x1="63.5" y1="53.34" x2="63.5" y2="49.53" width="0.4064" layer="20"/>
+<wire x1="54.61" y1="59.69" x2="54.61" y2="52.07" width="0.4064" layer="20"/>
+<wire x1="54.61" y1="52.07" x2="63.5" y2="52.07" width="0.4064" layer="20"/>
+<wire x1="63.5" y1="52.07" x2="63.5" y2="49.53" width="0.4064" layer="20"/>
 <wire x1="63.5" y1="49.53" x2="100.33" y2="49.53" width="0.4064" layer="20"/>
 <wire x1="100.33" y1="49.53" x2="100.33" y2="29.21" width="0.4064" layer="20"/>
 <wire x1="100.33" y1="29.21" x2="64.77" y2="29.21" width="0.4064" layer="20"/>
-<wire x1="64.77" y1="29.21" x2="64.77" y2="25.4" width="0.4064" layer="20"/>
-<wire x1="64.77" y1="25.4" x2="54.61" y2="25.4" width="0.4064" layer="20"/>
-<wire x1="54.61" y1="25.4" x2="54.61" y2="17.78" width="0.4064" layer="20"/>
+<wire x1="64.77" y1="29.21" x2="64.77" y2="26.67" width="0.4064" layer="20"/>
+<wire x1="64.77" y1="26.67" x2="54.61" y2="26.67" width="0.4064" layer="20"/>
+<wire x1="54.61" y1="26.67" x2="54.61" y2="17.78" width="0.4064" layer="20"/>
 <wire x1="54.61" y1="17.78" x2="-1.27" y2="17.78" width="0.4064" layer="20"/>
 <wire x1="-1.27" y1="17.78" x2="-1.27" y2="59.69" width="0.4064" layer="20"/>
@@
 <wire x1="62.23" y1="40.64" x2="60.96" y2="40.64" width="0.4064" layer="16"/>
 <wire x1="66.04" y1="40.64" x2="60.96" y2="40.64" width="0.4064" layer="16"/>
-<wire x1="40.64" y1="40.64" x2="39.37" y2="40.64" width="0.4064" layer="16"/>
-<wire x1="39.37" y1="40.64" x2="39.37" y2="35.56" width="0.4064" layer="16"/>
-<wire x1="39.37" y1="35.56" x2="21.59" y2="35.56" width="0.4064" layer="16"/>
+<wire x1="40.64" y1="40.64" x2="38.1" y2="40.64" width="0.4064" layer="16"/>
+<wire x1="38.1" y1="40.64" x2="38.1" y2="35.56" width="0.4064" layer="16"/>
+<wire x1="38.1" y1="35.56" x2="21.59" y2="35.56" width="0.4064" layer="16"/>
 <wire x1="21.59" y1="35.56" x2="21.59" y2="38.1" width="0.4064" layer="16"/>
 <wire x1="21.59" y1="38.1" x2="19.05" y2="38.1" width="0.4064" layer="16"/>
@@
 <contactref element="U1" pad="19"/>
 <wire x1="19.05" y1="33.02" x2="44.45" y2="33.02" width="0.4064" layer="16"/>
-<wire x1="45.72" y1="36.83" x2="45.72" y2="38.1" width="0.4064" layer="16"/>
-<wire x1="44.45" y1="33.02" x2="44.45" y2="35.56" width="0.4064" layer="16"/>
-<wire x1="44.45" y1="35.56" x2="45.72" y2="35.56" width="0.4064" layer="16"/>
-<wire x1="45.72" y1="35.56" x2="45.72" y2="38.1" width="0.4064" layer="16"/>
+<wire x1="44.45" y1="33.02" x2="44.45" y2="38.1" width="0.4064" layer="16"/>
+<wire x1="44.45" y1="38.1" x2="45.72" y2="38.1" width="0.4064" layer="16"/>
 </signal>
 <signal name="N$2">
@@
 <contactref element="U1" pad="18"/>
 <wire x1="19.05" y1="30.48" x2="45.72" y2="30.48" width="0.4064" layer="16"/>
-<wire x1="45.72" y1="30.48" x2="45.72" y2="34.29" width="0.4064" layer="16"/>
-<wire x1="45.72" y1="34.29" x2="50.8" y2="34.29" width="0.4064" layer="16"/>
-<wire x1="50.8" y1="34.29" x2="50.8" y2="38.1" width="0.4064" layer="16"/>
+<wire x1="45.72" y1="30.48" x2="45.72" y2="35.56" width="0.4064" layer="16"/>
+<wire x1="45.72" y1="35.56" x2="50.8" y2="35.56" width="0.4064" layer="16"/>
+<wire x1="50.8" y1="35.56" x2="50.8" y2="38.1" width="0.4064" layer="16"/>
 </signal>
 <signal name="N$7">
@@
 <wire x1="19.05" y1="27.94" x2="48.26" y2="27.94" width="0.4064" layer="16"/>
 <wire x1="58.42" y1="38.1" x2="60.96" y2="38.1" width="0.4064" layer="16"/>
-<wire x1="58.42" y1="31.75" x2="48.26" y2="31.75" width="0.4064" layer="16"/>
-<wire x1="48.26" y1="31.75" x2="48.26" y2="27.94" width="0.4064" layer="16"/>
-<wire x1="58.42" y1="31.75" x2="58.42" y2="38.1" width="0.4064" layer="16"/>
+<wire x1="58.42" y1="33.02" x2="48.26" y2="33.02" width="0.4064" layer="16"/>
+<wire x1="48.26" y1="33.02" x2="48.26" y2="27.94" width="0.4064" layer="16"/>
+<wire x1="58.42" y1="33.02" x2="58.42" y2="38.1" width="0.4064" layer="16"/>
 </signal>
 <signal name="N$9">
@@
 <contactref element="U1" pad="15"/>
 <wire x1="19.05" y1="22.86" x2="49.53" y2="22.86" width="0.4064" layer="16"/>
-<wire x1="49.53" y1="22.86" x2="49.53" y2="30.48" width="0.4064" layer="16"/>
-<wire x1="49.53" y1="30.48" x2="59.69" y2="30.48" width="0.4064" layer="16"/>
-<wire x1="59.69" y1="30.48" x2="59.69" y2="35.56" width="0.4064" layer="16"/>
+<wire x1="49.53" y1="22.86" x2="49.53" y2="31.75" width="0.4064" layer="16"/>
+<wire x1="49.53" y1="31.75" x2="59.69" y2="31.75" width="0.4064" layer="16"/>
+<wire x1="59.69" y1="31.75" x2="59.69" y2="35.56" width="0.4064" layer="16"/>
 <wire x1="59.69" y1="35.56" x2="66.04" y2="35.56" width="0.4064" layer="16"/>
 <wire x1="66.04" y1="35.56" x2="66.04" y2="38.1" width="0.4064" layer="16"/>
@@
 <wire x1="13.97" y1="22.86" x2="13.97" y2="19.05" width="0.4064" layer="16"/>
 <wire x1="13.97" y1="19.05" x2="53.34" y2="19.05" width="0.4064" layer="16"/>
-<wire x1="53.34" y1="19.05" x2="53.34" y2="26.67" width="0.4064" layer="16"/>
+<wire x1="53.34" y1="19.05" x2="53.34" y2="27.94" width="0.4064" layer="16"/>
 <wire x1="63.5" y1="31.75" x2="73.66" y2="31.75" width="0.4064" layer="16"/>
 <wire x1="73.66" y1="31.75" x2="73.66" y2="35.56" width="0.4064" layer="16"/>
@@
 <wire x1="78.74" y1="35.56" x2="78.74" y2="38.1" width="0.4064" layer="16"/>
 <wire x1="78.74" y1="38.1" x2="81.28" y2="38.1" width="0.4064" layer="16"/>
-<wire x1="53.34" y1="26.67" x2="63.5" y2="26.67" width="0.4064" layer="16"/>
-<wire x1="63.5" y1="26.67" x2="63.5" y2="31.75" width="0.4064" layer="16"/>
+<wire x1="53.34" y1="27.94" x2="63.5" y2="27.94" width="0.4064" layer="16"/>
+<wire x1="63.5" y1="27.94" x2="63.5" y2="31.75" width="0.4064" layer="16"/>
 </signal>
 <signal name="N$11">
@@
 <wire x1="72.39" y1="36.83" x2="76.2" y2="36.83" width="0.4064" layer="16"/>
 <wire x1="76.2" y1="36.83" x2="76.2" y2="38.1" width="0.4064" layer="16"/>
-<wire x1="62.23" y1="27.94" x2="52.07" y2="27.94" width="0.4064" layer="16"/>
-<wire x1="52.07" y1="27.94" x2="52.07" y2="20.32" width="0.4064" layer="16"/>
-<wire x1="62.23" y1="27.94" x2="62.23" y2="33.02" width="0.4064" layer="16"/>
+<wire x1="62.23" y1="29.21" x2="52.07" y2="29.21" width="0.4064" layer="16"/>
+<wire x1="52.07" y1="29.21" x2="52.07" y2="20.32" width="0.4064" layer="16"/>
+<wire x1="62.23" y1="29.21" x2="62.23" y2="33.02" width="0.4064" layer="16"/>
 </signal>
 <signal name="N$12">
@@
 <wire x1="16.51" y1="27.94" x2="16.51" y2="29.21" width="0.4064" layer="16"/>
 <wire x1="16.51" y1="29.21" x2="46.99" y2="29.21" width="0.4064" layer="16"/>
-<wire x1="55.88" y1="33.02" x2="46.99" y2="33.02" width="0.4064" layer="16"/>
-<wire x1="46.99" y1="33.02" x2="46.99" y2="29.21" width="0.4064" layer="16"/>
-<wire x1="55.88" y1="33.02" x2="55.88" y2="38.1" width="0.4064" layer="16"/>
+<wire x1="55.88" y1="34.29" x2="46.99" y2="34.29" width="0.4064" layer="16"/>
+<wire x1="46.99" y1="34.29" x2="46.99" y2="29.21" width="0.4064" layer="16"/>
+<wire x1="55.88" y1="34.29" x2="55.88" y2="38.1" width="0.4064" layer="16"/>
 </signal>
 <signal name="N$13">
@@
 <wire x1="60.96" y1="34.29" x2="71.12" y2="34.29" width="0.4064" layer="16"/>
 <wire x1="71.12" y1="34.29" x2="71.12" y2="38.1" width="0.4064" layer="16"/>
-<wire x1="60.96" y1="29.21" x2="50.8" y2="29.21" width="0.4064" layer="16"/>
-<wire x1="50.8" y1="29.21" x2="50.8" y2="21.59" width="0.4064" layer="16"/>
-<wire x1="60.96" y1="29.21" x2="60.96" y2="34.29" width="0.4064" layer="16"/>
+<wire x1="60.96" y1="30.48" x2="50.8" y2="30.48" width="0.4064" layer="16"/>
+<wire x1="50.8" y1="30.48" x2="50.8" y2="21.59" width="0.4064" layer="16"/>
+<wire x1="60.96" y1="30.48" x2="60.96" y2="34.29" width="0.4064" layer="16"/>
 </signal>
 <signal name="N$19">
@@
 <vertex x="-1.27" y="59.69"/>
 <vertex x="54.61" y="59.69"/>
-<vertex x="54.61" y="53.34"/>
-<vertex x="63.5" y="53.34"/>
+<vertex x="54.61" y="52.07"/>
+<vertex x="63.5" y="52.07"/>
 <vertex x="63.5" y="49.53"/>
 <vertex x="100.33" y="49.53"/>
 <vertex x="100.33" y="29.21"/>
 <vertex x="64.77" y="29.21"/>
-<vertex x="64.77" y="25.4"/>
-<vertex x="54.61" y="25.4"/>
+<vertex x="64.77" y="26.67"/>
+<vertex x="54.61" y="26.67"/>
 <vertex x="54.61" y="17.78"/>
 <vertex x="-1.27" y="17.78"/>
@@
 <vertex x="-1.27" y="59.69"/>
 <vertex x="54.61" y="59.69"/>
-<vertex x="54.61" y="53.34"/>
-<vertex x="63.5" y="53.34"/>
+<vertex x="54.61" y="52.07"/>
+<vertex x="63.5" y="52.07"/>
 <vertex x="63.5" y="49.53"/>
 <vertex x="100.33" y="49.53"/>
 <vertex x="100.33" y="29.21"/>
 <vertex x="64.77" y="29.21"/>
-<vertex x="64.77" y="25.4"/>
-<vertex x="54.61" y="25.4"/>
+<vertex x="64.77" y="26.67"/>
+<vertex x="54.61" y="26.67"/>
 <vertex x="54.61" y="17.78"/>
 <vertex x="-1.27" y="17.78"/>
